File: hardware/jackboard_singlelayer/drumcore_jackboard_singlelayer.kicad_pcb (KiCad board)
At the start: 2 copper layers, 184 x 57.5 mm, 58 parts, among them J1 PAD1_TRS_6.35MM, J2 PAD2_TRS_6.35MM, J3 PAD3_TRS_6.35MM, J4 PAD4_TRS_6.35MM, J5 PAD5_TRS_6.35MM, J6 PAD6_TRS_6.35MM, J7 PAD7_TRS_6.35MM, J8 PAD8_TRS_6.35MM, U1 HC4067_CHANNELS, U2 HC4067_CTRL

Commit message: Jackboard single-layer: grampo duplo com 1N4148, 1k em serie, 4,7k no SIG e trilhas de 0,8mm
Protecao por canal revisada para usar 1N4148 (o BAT85 e' dificil de
achar aqui):
- R1-R16 (serie) de 100R para 1k, pra limitar a corrente que passa pelo
  grampo, ja' que o 1N4148 grampeia ~0,4V mais alto que o Schottky.
- D1-D16 trocados de BAT85 para 1N4148 (mesma posicao, catodo no sinal,
  anodo no GND).
- Novos D17-D32 (1N4148, anodo no MUX_Cn, catodo no +3V3): grampeiam os
  picos acima da alimentacao do ADC, que antes nao tinham protecao na
  placa. Ficam em pe embaixo da placa do MUX, um sobre cada pino de canal
  do U1, com a trilha de +3V3 estendida ate o C15.
- Novo R33 (4,7k do MUX_SIG pro GND): descarrega a capacitancia do SIG
  entre um canal e outro (o breakout do CD4067 so' tem 10k no EN).

Trilhas passaram de 0,5mm para 0,8mm: a primeira placa corroida mostrou
que 0,5mm ficava fino demais na transferencia termica. Simulacao de folga
antes da mudanca: pior caso 0,93mm (C1 ao lado do C2); 1,2mm ja' violava
a folga de 0,65mm.

Ponte de GND por cima do U2 (pino 3 ao pino 1): com a trilha de +3V3
estendida, o pino 3 ficava com uma so' ponte de alivio termico e o KiCad
o deixava sem conexao.

DRC: 0 itens sem conexao, 0 folga/curto, esquematico e PCB batendo. ERC:
0 erros. PDFs de transferencia termica (placa unica e 4 por A4)
regenerados em fab/.

Co-Authored-By: Claude Opus 5.5 (1M context) <noreply@anthropic.com>
Parts:
- added D17: 1N4148, Diode_THT:D_DO-35_SOD27_P7.62mm_Horizontal, F.Cu at (166.2, 78.1)
- added D18: 1N4148, Diode_THT:D_DO-35_SOD27_P7.62mm_Horizontal, F.Cu at (163.6, 78.1)
- added D19: 1N4148, Diode_THT:D_DO-35_SOD27_P7.62mm_Horizontal, F.Cu at (161.1, 78.1)
- added D20: 1N4148, Diode_THT:D_DO-35_SOD27_P7.62mm_Horizontal, F.Cu at (158.6, 78.1)
- added D21: 1N4148, Diode_THT:D_DO-35_SOD27_P7.62mm_Horizontal, F.Cu at (156.0, 78.1)
- added D22: 1N4148, Diode_THT:D_DO-35_SOD27_P7.62mm_Horizontal, F.Cu at (153.5, 78.1)
- added D23: 1N4148, Diode_THT:D_DO-35_SOD27_P7.62mm_Horizontal, F.Cu at (150.9, 78.1)
- added D24: 1N4148, Diode_THT:D_DO-35_SOD27_P7.62mm_Horizontal, F.Cu at (148.4, 78.1)
- added D25: 1N4148, Diode_THT:D_DO-35_SOD27_P7.62mm_Horizontal, F.Cu at (145.9, 78.1)
- added D26: 1N4148, Diode_THT:D_DO-35_SOD27_P7.62mm_Horizontal, F.Cu at (143.3, 78.1)
- added D27: 1N4148, Diode_THT:D_DO-35_SOD27_P7.62mm_Horizontal, F.Cu at (140.8, 78.1)
- added D28: 1N4148, Diode_THT:D_DO-35_SOD27_P7.62mm_Horizontal, F.Cu at (138.2, 78.1)
- added D29: 1N4148, Diode_THT:D_DO-35_SOD27_P7.62mm_Horizontal, F.Cu at (135.7, 78.1)
- added D30: 1N4148, Diode_THT:D_DO-35_SOD27_P7.62mm_Horizontal, F.Cu at (133.2, 78.1)
- added D31: 1N4148, Diode_THT:D_DO-35_SOD27_P7.62mm_Horizontal, F.Cu at (130.6, 78.1)
- added D32: 1N4148, Diode_THT:D_DO-35_SOD27_P7.62mm_Horizontal, F.Cu at (128.1, 78.1)
- added R33: 4.7k, Resistor_THT:R_Axial_DIN0207_L6.3mm_D2.5mm_P7.62mm_Horizontal, F.Cu at (121.2, 74.2)
- D1, D10, D11, D12, D13, D14, D15, D16, D2, D3, D4, D5, D6, D7, D8, D9: value BAT85 -> 1N4148
- R1, R10, R11, R12, R13, R14, R15, R16, R2, R3, R4, R5, R6, R7, R8, R9: value 100R -> 1k
Routing:
- net /+3V3: track 104.4 -> 128.7 mm
- net /MUX_SIG: track 0.00 -> 17.1 mm
- net /GND: track 0.00 -> 10.1 mm
- net /MUX_C14: track 85.3 -> 89.4 mm
- net /MUX_C15: track 98.1 -> 101.8 mm
- net /MUX_C9: track 44.7 -> 48.4 mm
- net /MUX_C8: track 33.0 -> 36.8 mm
- net /MUX_C7: track 38.4 -> 42.1 mm
- net /MUX_C5: track 55.8 -> 59.5 mm
- net /MUX_C4: track 43.9 -> 47.7 mm
- net /MUX_C3: track 73.2 -> 76.9 mm
- net /MUX_C13: track 79.5 -> 83.3 mm
- net /MUX_C12: track 68.1 -> 71.8 mm
- net /MUX_C10: track 50.4 -> 54.2 mm
- net /MUX_C1: track 92.0 -> 95.8 mm
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