File: hardware/jackboard_singlelayer/drumcore_jackboard_singlelayer.kicad_sch (KiCad schematic)
At the start: 58 parts, among them J1 PAD1_TRS_6.35MM, J2 PAD2_TRS_6.35MM, J3 PAD3_TRS_6.35MM, J4 PAD4_TRS_6.35MM, J5 PAD5_TRS_6.35MM, J6 PAD6_TRS_6.35MM, J7 PAD7_TRS_6.35MM, J8 PAD8_TRS_6.35MM, U1 HC4067_CHANNELS, U2 HC4067_CTRL

Commit message: Jackboard single-layer: grampo duplo com 1N4148, 1k em serie, 4,7k no SIG e trilhas de 0,8mm
Protecao por canal revisada para usar 1N4148 (o BAT85 e' dificil de
achar aqui):
- R1-R16 (serie) de 100R para 1k, pra limitar a corrente que passa pelo
  grampo, ja' que o 1N4148 grampeia ~0,4V mais alto que o Schottky.
- D1-D16 trocados de BAT85 para 1N4148 (mesma posicao, catodo no sinal,
  anodo no GND).
- Novos D17-D32 (1N4148, anodo no MUX_Cn, catodo no +3V3): grampeiam os
  picos acima da alimentacao do ADC, que antes nao tinham protecao na
  placa. Ficam em pe embaixo da placa do MUX, um sobre cada pino de canal
  do U1, com a trilha de +3V3 estendida ate o C15.
- Novo R33 (4,7k do MUX_SIG pro GND): descarrega a capacitancia do SIG
  entre um canal e outro (o breakout do CD4067 so' tem 10k no EN).

Trilhas passaram de 0,5mm para 0,8mm: a primeira placa corroida mostrou
que 0,5mm ficava fino demais na transferencia termica. Simulacao de folga
antes da mudanca: pior caso 0,93mm (C1 ao lado do C2); 1,2mm ja' violava
a folga de 0,65mm.

Ponte de GND por cima do U2 (pino 3 ao pino 1): com a trilha de +3V3
estendida, o pino 3 ficava com uma so' ponte de alivio termico e o KiCad
o deixava sem conexao.

DRC: 0 itens sem conexao, 0 folga/curto, esquematico e PCB batendo. ERC:
0 erros. PDFs de transferencia termica (placa unica e 4 por A4)
regenerados em fab/.

Co-Authored-By: Claude Opus 5.5 (1M context) <noreply@anthropic.com>
Parts:
- added D17, D18, D19, D20, D21, D22, D23, D24, D25, D26, D27, D28, D29, D30, D31, D32: 1N4148, Diode_THT:D_DO-35_SOD27_P7.62mm_Horizontal, symbol Diode:1N4148
- added R33: 4.7k, Resistor_THT:R_Axial_DIN0207_L6.3mm_D2.5mm_P7.62mm_Horizontal, symbol Device:R
- D1, D10, D11, D12, D13, D14, D15, D16, D2, D3, D4, D5, D6, D7, D8, D9: value BAT85 -> 1N4148; symbol Diode:BAT85 -> Diode:1N4148
- R1, R10, R11, R12, R13, R14, R15, R16, R2, R3, R4, R5, R6, R7, R8, R9: value 100R -> 1k
Connections:
- net +3V3: now also D17.1 (K), D18.1 (K), D19.1 (K), D20.1 (K), D21.1 (K), D22.1 (K), D23.1 (K), D24.1 (K), D25.1 (K), D26.1 (K), D27.1 (K), D28.1 (K), D29.1 (K), D30.1 (K), D31.1 (K), D32.1 (K)
- net GND: now also R33.2
- net MUX_C0: now also D17.2 (A)
- net MUX_C1: now also D18.2 (A)
- net MUX_C10: now also D27.2 (A)
- net MUX_C11: now also D28.2 (A)
- net MUX_C12: now also D29.2 (A)
- net MUX_C13: now also D30.2 (A)
- net MUX_C14: now also D31.2 (A)
- net MUX_C15: now also D32.2 (A)
- net MUX_C2: now also D19.2 (A)
- net MUX_C3: now also D20.2 (A)
- net MUX_C4: now also D21.2 (A)
- net MUX_C5: now also D22.2 (A)
- net MUX_C6: now also D23.2 (A)
- net MUX_C7: now also D24.2 (A)
- net MUX_C8: now also D25.2 (A)
- net MUX_C9: now also D26.2 (A)
- net MUX_SIG: now also R33.1
